File: Snaefellsjoekull_panMonoChannel/Snaefellsjoekull_panMonoChannel.kicad_pcb (KiCad board)
At the start: 2 copper layers, 15 x 100 mm, 9 parts, among them J1 AudioJack2_SwitchT, J2 Bus Connector

Commit message: Potentiometer fixed
Parts:
- RV1: value 10k_log -> 10k
Connections:
- RV1 pad 1: GND -> Net-(J1-PadT)
- RV1 pad 3: Net-(J1-PadT) -> GND
Routing:
- net Net-(J1-PadT): track 63.1 -> 65.2 mm
